File: ECMEndstopPumpInterface/ECMEndstopPumpInterface.kicad_pcb (KiCad board)
At the start: 2 copper layers, 130.8 x 45.7 mm, 57 parts, among them J1 Endstop, J10 GPIOEndstop, J11 Endstop, J12 Endstop, J13 Load12, J14 Endstop, J15 Endstop, J16 Endstop, J17 Power, J18 Power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

Commit message: Adding Gerber files
Other:
- board text added: "ECM Pump and Endstop Interface Board https://github.com/tspspi/ecmendstopandpumpinterfacev1 (33c4680c2ffe952bb6c5bdeb57909ba8fada2b4d) https://www.tspi.at"
- board text removed: "ECM Pump and Endstop Interface Board https://github.com/tspspi/ecmendstopandpumpinterfacev1 () https://www.tspi.at"
